File: hardware/mimic0x/mimic00/mimic00.kicad_pcb (KiCad board)
At the start: 2 copper layers, 38 x 20 mm, 30 parts, among them J1 Conn_01x06, J2 Conn_01x06, J3 Conn_01x03, J5 Conn_01x05, U1 PY32F071C1BU6TR_DIY

Commit message: Add hybrid open-source licenses (CERN-OHL-S, GPLv3, MIT)
Other:
- board text added: "© 2026 K. TAKAGI CERN-OHL-S-2.0"
Changed lines of the file:
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@@
 	)
 	(paper "A4")
+	(title_block
+		(comment 1 "License: CERN-OHL-S-2.0")
+		(comment 2 "Copyright (C) 2026 TAKAGI Katsuyuki")
+		(comment 3 "Project: Analog Mimic")
+	)
 	(layers
 		(0 "F.Cu" signal)
@@
 		)
 	)
+	(gr_text "© 2026 K. TAKAGI\nCERN-OHL-S-2.0"
+		(at 155.238761 97.070847 0)
+		(layer "B.SilkS")
+		(effects
+			(font
+				(size 0.8 0.8)
+				(thickness 0.12)
+			)
+			(justify left bottom mirror)
+		)
+	)
