File: hardware/mimic0x/mimic01/mimic01.kicad_pcb (KiCad board)
At the start: 2 copper layers, 35.6 x 20 mm, 33 parts, among them J2 Conn_01x06, J3 Conn_01x03, J5 Conn_01x05, Q1 AO3401A, SW1 TS-1088-AR02016, U1 PY32F071C1BU6TR_DIY

Commit message: add input bias, vdd/2
Parts:
- added C10: 0.1uF, Capacitor_SMD:C_0402_1005Metric, F.Cu at (140.1, 96.7)
- added R15: 100k, Resistor_SMD:R_0402_1005Metric, F.Cu at (138.6, 98.2)
- added R3: 100k, Resistor_SMD:R_0402_1005Metric, F.Cu at (140.1, 97.7)
- R11, R12, R13: value 3.3k -> 10k
- moved R2 5.59 mm to (138.6, 96.2), turned to -90 degrees
- moved LED1 2.04 mm to (142.3, 99.0), turned to 90 degrees
- moved R14 0.77 mm to (143.3, 97.2)
Connections:
- R2 pad 2: GND -> Net-(C10-Pad1)
Routing:
- net Net-(C10-Pad1): track 0.00 -> 2.06 mm
- net /AIN: track 11.0 -> 9.99 mm
- net VCC: track 92.5 -> 93.3 mm
- net GND: vias 107 -> 111
Other:
- board text added: "26.10.25"
- board text removed: "26.5.22"

Commit message: changed: input bias voltage, VDD/2. pullup resistor value, 10k. silk texts. add OSHW logo
Parts:
- added REF**: OSHW-Logo2_9.8x8mm_SilkScreen, Symbol:OSHW-Logo2_9.8x8mm_SilkScreen, B.Cu at (152.5, 102.3)
Routing:
- net Net-(C10-Pad1): track 2.06 -> 3.07 mm
Other:
- board text added: "2026-10-25"
- board text added: "JPYYYYMM"
- board text removed: "26.10.25"

Commit message: Add OSHW certification  (JP000025)
Parts:
- removed the REF** at (152.5, 102.3)
- added REF**: OSHW-Certification-Mark-Stacked_8x7mm_SilkScreen, OSHW:OSHW-Certification-Mark-Stacked_8x7mm_SilkScreen, B.Cu at (152.5, 102.0)
Other:
- board text added: "2026-10-29"
- board text removed: "2026-10-25"
- board text removed: "JPYYYYMM"
